File: BS2103F_photo/BS2103F_photo.kicad_pcb (KiCad board)
At the start: 2 copper layers, 50 x 70 mm, 41 parts, among them J1 Vs, J2 Motors, J3 VccAndIN, Q1 BSJ300N10, Q2 BSJ300N10, Q3 BSJ300N10, Q4 BSJ300N10, U1 L7812, U2 TLP291, U3 TLP291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

Commit message: add PCBdata
Parts:
- added G***: LOGO, purin:LOGO, B.Cu at (150.0, 98.0)
- moved R14 1.52 mm to (156.2, 88.5)
- moved R20 1.52 mm to (156.2, 116.5)
- moved R13 1.33 mm to (156.2, 83.1)
- moved R19 1.33 mm to (156.2, 111.1)
Routing:
- net GND: track 0.00 -> 153.5 mm
- net Net-(C3-Pad1): track 0.00 -> 102.8 mm, vias 0 -> 2
- net 24V: track 0.00 -> 97.2 mm
- net Motor2: track 0.00 -> 83.0 mm
- net Motor1: track 0.00 -> 66.7 mm, vias 0 -> 2
- net Net-(R12-Pad2): track 0.00 -> 50.5 mm
- net PINGND: track 0.00 -> 34.1 mm
- net Net-(R10-Pad2): track 0.00 -> 29.8 mm
- net 5V: track 0.00 -> 23.6 mm
- net ShutDown: track 0.00 -> 23.5 mm
- net IN2: track 0.00 -> 20.1 mm
- net IN1: track 0.00 -> 11.9 mm
- net Net-(Q1-Pad1): track 0.00 -> 11.4 mm
- net Net-(Q3-Pad1): track 0.00 -> 11.4 mm
- net Net-(R11-Pad2): track 0.00 -> 10.8 mm
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- added copper zone on B.Cu, net GND
- added copper zone on F.Cu, net GND
Other:
- net class Power: trace_width 1.5 -> 1.2
- board text added: "0.1uF"
- board text added: "10"
- board text added: "100"
- board text added: "1000uF"
- board text added: "100k"
- board text added: "100uF"
- board text added: "10k"
- board text added: "24V"
- board text added: "5V"
- board text added: "7812"
- board text added: "Diode"
- board text added: "GND"
- board text added: "IN1"
- board text added: "IN2"
- board text added: "IR2104"
- board text added: "LED"
- board text added: "Motor"
- board text added: "RSJ300N10"
- board text added: "Shutdown"
- board text added: "TLP291"
- board text added: "ei24VNchMD 2018/11/22"
- board text added: "pinGND"
